File: etherrail-control-1000.kicad_sch (KiCad schematic)
At the start: 33 parts, among them J1 Conn_02x04_Counter_Clockwise, J2 Conn_01x04, U1 AMS1117-3.3, U2 ESP32-C3, Y2 Crystal_GND24

Commit message: Add PCB
Parts:
- removed J1: Conn_02x04_Counter_Clockwise, Connector_PinSocket_2.54mm:PinSocket_2x04_P2.54mm_Vertical, symbol Connector_Generic:Conn_02x04_Counter_Clockwise
- added J1: Conn_02x04_Odd_Even, Connector_PinHeader_2.54mm:PinHeader_2x04_P2.54mm_Vertical, symbol Connector_Generic:Conn_02x04_Odd_Even
- J2: footprint (none) -> Connector_PinHeader_1.00mm:PinHeader_1x04_P1.00mm_Vertical
- U3: footprint (none) -> Package_DFN_QFN:DFN-8-1EP_3x3mm_P0.65mm_EP1.55x2.4mm
- Y2: footprint (none) -> Crystal:Crystal_SMD_3225-4Pin_3.2x2.5mm
Connections:
- net Controller Power: now also U2.31 (VDDA), U2.32 (VDDA)
- net GND: now also C7.2, C8.2
- net Light Common (+): now also J1.4 (Pin_4)
- net Light Front (-): now also J1.6 (Pin_6)
- net Light Rear (-): now also J1.3 (Pin_3)
- net Motor Controlling Direction: now also U2.23 (SPID/GPIO16); no longer U2.24 (SPIQ/GPIO17)
- net Motor Controlling PWM: now also U2.24 (SPIQ/GPIO17); no longer U2.23 (SPID/GPIO16)
- net Motor Negative: now also J1.8 (Pin_8)
- net Motor Positive: now also J1.1 (Pin_1)
- net Power Pickup Left: now also J1.7 (Pin_7)
- net Power Pickup Right: now also J1.2 (Pin_2)
Other:
- moved on the sheet: C7, C8

Commit message: Fix 10uF cap footprint
Parts:
- C4: footprint Capacitor_SMD:C_0201_0603Metric -> Capacitor_SMD:C_0402_1005Metric
Changed lines of the file:
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@@
       (effects (font (size 1.27 1.27)) hide)
     )
-    (pin "2")
-    (pin "1")
+    (pin "1")
+    (pin "2")
     (instances
       (project "etherrail-control-1000"
@@
       (effects (font (size 1.27 1.27)) hide)
     )
-    (pin "2")
-    (pin "1")
+    (pin "1")
+    (pin "2")
     (instances
       (project "etherrail-control-1000"
@@
       (effects (font (size 1.27 1.27)) hide)
     )
-    (pin "2")
-    (pin "1")
+    (pin "1")
+    (pin "2")
     (instances
       (project "etherrail-control-1000"
@@
       (effects (font (size 1.27 1.27)) hide)
     )
-    (pin "2")
-    (pin "1")
+    (pin "1")
+    (pin "2")
     (instances
       (project "etherrail-control-1000"
@@
       (effects (font (size 1.27 1.27)) hide)
     )
-    (pin "2")
-    (pin "1")
+    (pin "1")
+    (pin "2")
     (instances
       (project "etherrail-control-1000"
@@
       (effects (font (size 1.27 1.27)) hide)
     )
-    (pin "2")
-    (pin "1")
+    (pin "1")
+    (pin "2")
     (instances
       (project "etherrail-control-1000"
@@
       (effects (font (size 1.27 1.27)) hide)
     )
-    (pin "2")
-    (pin "1")
-    (pin "8")
+    (pin "1")
+    (pin "2")
+    (pin "3")
+    (pin "4")
     (pin "5")
-    (pin "4")
     (pin "6")
     (pin "7")
-    (pin "3")
+    (pin "8")
     (instances
       (project "etherrail-control-1000"
@@
       (effects (font (size 1.27 1.27)) hide)
     )
-    (pin "2")
-    (pin "1")
+    (pin "1")
+    (pin "2")
     (instances
       (project "etherrail-control-1000"
@@
       (effects (font (size 1.27 1.27)) hide)
     )
-    (pin "8")
+    (pin "1")
+    (pin "2")
     (pin "3")
-    (pin "7")
     (pin "4")
     (pin "5")
     (pin "6")
-    (pin "2")
-    (pin "1")
+    (pin "7")
+    (pin "8")
     (instances
       (project "etherrail-control-1000"
@@
       (effects (font (size 1.27 1.27)) (justify left))
     )
-    (property "Footprint" "Capacitor_SMD:C_0201_0603Metric" (at 102.5652 67.31 0)
+    (property "Footprint" "Capacitor_SMD:C_0402_1005Metric" (at 102.5652 67.31 0)
       (effects (font (size 1.27 1.27)) hide)
     )
@@
       (effects (font (size 1.27 1.27)) hide)
     )
-    (pin "2")
-    (pin "1")
+    (pin "1")
+    (pin "2")
     (instances
       (project "etherrail-control-1000"
@@
       (effects (font (size 1.27 1.27)) hide)
     )
-    (pin "2")
-    (pin "1")
+    (pin "1")
+    (pin "2")
     (instances
       (project "etherrail-control-1000"
@@
       (effects (font (size 1.27 1.27)) hide)
     )
-    (pin "2")
-    (pin "1")
+    (pin "1")
+    (pin "2")
     (instances
       (project "etherrail-control-1000"
@@
       (effects (font (size 1.27 1.27)) hide)
     )
-    (pin "2")
-    (pin "1")
+    (pin "1")
+    (pin "2")
     (instances
       (project "etherrail-control-1000"
@@
       (effects (font (size 1.27 1.27)) hide)
     )
+    (pin "1")
+    (pin "2")
+    (pin "3")
     (pin "4")
-    (pin "1")
-    (pin "3")
-    (pin "2")
     (instances
       (project "etherrail-control-1000"
@@
       (effects (font (size 1.27 1.27)) hide)
     )
-    (pin "2")
-    (pin "1")
+    (pin "1")
+    (pin "2")
     (instances
       (project "etherrail-control-1000"
@@
     )
     (pin "1")
-    (pin "25")
-    (pin "3")
+    (pin "10")
     (pin "11")
-    (pin "21")
-    (pin "24")
-    (pin "4")
-    (pin "9")
-    (pin "31")
-    (pin "26")
-    (pin "29")
-    (pin "33")
-    (pin "28")
-    (pin "27")
-    (pin "30")
-    (pin "7")
     (pin "12")
-    (pin "5")
     (pin "13")
     (pin "14")
     (pin "15")
     (pin "16")
-    (pin "32")
     (pin "17")
     (pin "18")
     (pin "19")
     (pin "2")
+    (pin "20")
+    (pin "21")
+    (pin "22")
     (pin "23")
-    (pin "22")
-    (pin "20")
+    (pin "24")
+    (pin "25")
+    (pin "26")
+    (pin "27")
+    (pin "28")
+    (pin "29")
+    (pin "30")
+    (pin "31")
+    (pin "33")
+    (pin "4")
+    (pin "5")
+    (pin "6")
+    (pin "7")
     (pin "8")
-    (pin "6")
-    (pin "10")
+    (pin "9")
+    (pin "3")
+    (pin "32")
     (instances
       (project "etherrail-control-1000"
@@
       (effects (font (size 1.27 1.27)) hide)
     )
-    (pin "2")
-    (pin "1")
+    (pin "1")
+    (pin "2")
     (instances
       (project "etherrail-control-1000"
@@
       (effects (font (size 1.27 1.27)) hide)
     )
-    (pin "2")
-    (pin "1")
+    (pin "1")
+    (pin "2")
     (instances
       (project "etherrail-control-1000"
@@
       (effects (font (size 1.27 1.27)) hide)
     )
-    (pin "2")
-    (pin "1")
+    (pin "1")
+    (pin "2")
     (instances
       (project "etherrail-control-1000"
@@
       (effects (font (size 1.27 1.27)) hide)
     )
-    (pin "2")
+    (pin "1")
+    (pin "2")
+    (pin "3")
     (pin "4")
-    (pin "3")
-    (pin "1")
-    (instances
-      (project "etherrail-control-1000"
+    (instances
+      (project "etherrail-control-1000"
